File: CheckPoint1/KiCAD/probando/probando.kicad_sch (KiCad schematic)
At the start: 10 parts, among them J1 Conn_01x02, Q2 BC547, Q3 BC557, Q4 BC557, Q5 BC547, Q6 BC547, Q7 BC547, Q8 BC547, Q9 BC547

Commit message: kicad 1
Parts:
- added JP1: Jumper_2_Bridged, symbol Jumper:Jumper_2_Bridged
- R3: renamed from R1; value R -> 4k4
Connections:
- net GND: now also Q6.3 (E), Q7.3 (E)
- net at Q4.1 (C): now also Q2.1 (C), Q3.2 (B), Q4.2 (B)
- net at Q3.1 (C): now also Q5.1 (C)
- net at Q6.1 (C): now also JP1.1 (A); no longer Q5.3 (E)
- net at Q6.2 (B): now also Q7.1 (C), Q7.2 (B), R3.2
- net at Q2.3 (E): now also Q5.3 (E), JP1.2 (B)
Other:
- moved on the sheet: Q6, Q7, R3
