File: CheckPoint1/KiCad/esquematico/esquematico.kicad_sch (KiCad schematic)
At the start: 33 parts, among them J1 Conn_01x02, J2 Conn_01x02, Q10 TIP32A, Q2 BC547, Q3 BC557, Q4 BC557, Q5 BC547, Q6 BC547, Q7 BC547, Q8 BC547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

Commit message: new changes
Parts:
- renumbered Q5 to Q1, Q10 to Q5, R1 to R10, R2 to R11, R4 to R6
Changed lines of the file:
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@@
 		(date "2026-04-10")
 		(company "FIUBA - TA138")
-		(comment 1 "Lautaro, García Vitale - Padrón: 110028")
-		(comment 2 "Santiago Manuel, Cabrera - Padrón: 110445")
-		(comment 3 "Francisco Javier, Moya - Padrón: 109899")
+		(comment 1 "Lautaro García Vitale - Padrón: 110028")
+		(comment 2 "Santiago Manuel Cabrera - Padrón: 110445")
+		(comment 3 "Francisco Javier Moya - Padrón: 109899")
 		(comment 4 "Integrantes:")
 	)
@@
 		(in_pos_files yes)
 		(dnp no)
-		(property "Reference" "Q10"
+		(property "Reference" "Q5"
 			(at 186.69 60.9599 0)
 			(show_name no)
@@
 			(project "esquematico"
 				(path "/70816206-2001-4ff4-9567-5d4a4798dbfa"
-					(reference "Q10")
+					(reference "Q5")
 					(unit 1)
 				)
@@
 		(in_pos_files yes)
 		(dnp no)
-		(property "Reference" "Q5"
+		(property "Reference" "Q1"
 			(at 120.65 88.8999 0)
 			(show_name no)
@@
 			(project "esquematico"
 				(path "/70816206-2001-4ff4-9567-5d4a4798dbfa"
-					(reference "Q5")
+					(reference "Q1")
 					(unit 1)
 				)
@@
 		(dnp no)
 		(fields_autoplaced yes)
-		(property "Reference" "R2"
+		(property "Reference" "R11"
 			(at 116.84 128.2699 0)
 			(show_name no)
@@
 			(project "esquematico"
 				(path "/70816206-2001-4ff4-9567-5d4a4798dbfa"
-					(reference "R2")
+					(reference "R11")
 					(unit 1)
 				)
@@
 		(dnp no)
 		(fields_autoplaced yes)
-		(property "Reference" "R4"
+		(property "Reference" "R6"
 			(at 107.95 53.3399 0)
 			(show_name no)
@@
 			(project "esquematico"
 				(path "/70816206-2001-4ff4-9567-5d4a4798dbfa"
-					(reference "R4")
+					(reference "R6")
 					(unit 1)
 				)
@@
 		(dnp no)
 		(fields_autoplaced yes)
-		(property "Reference" "R1"
+		(property "Reference" "R10"
 			(at 77.47 128.2699 0)
 			(show_name no)
@@
 			(project "esquematico"
 				(path "/70816206-2001-4ff4-9567-5d4a4798dbfa"
-					(reference "R1")
+					(reference "R10")
 					(unit 1)
 				)
