File: Checkpoint2/KiCAD/Diseño/Diseño.kicad_pcb (KiCad board)
At the start: 2 copper layers, 120 x 85 mm, 36 parts, among them J1 Conn_01x02, Q1 BC547, Q2 BC547, Q3 BC557, Q4 BC557, Q5 BC547, Q6 TIP32A, Q7 BC547, Q8 BC547, Q9 BC547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

Commit message: con 40n compensa este hijo de puta
Routing:
- net Net-(Q2-C): track 27.5 -> 38.2 mm
- net Net-(J_LC1-A): track 0.00 -> 6.57 mm
- net /Vo: track 22.6 -> 25.8 mm
- net Net-(U2A-+): track 13.4 -> 15.7 mm
Changed lines of the file:
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@@
+	)
+	(segment
+		(start 157 110)
+		(end 160.19 110)
+		(width 0.2)
+		(layer "F.Cu")
+		(net "/Vo")
 	)
 	(segment
@@
 		(start 133 88)
 		(end 128.46 88)
+		(width 0.2)
+		(layer "F.Cu")
+		(net "Net-(Q2-C)")
+	)
+	(segment
+		(start 136 97.46)
+		(end 136 91)
 		(width 0.2)
 		(layer "F.Cu")
@@
 	)
 	(segment
+		(start 136 91)
+		(end 133 88)
+		(width 0.2)
+		(layer "F.Cu")
+		(net "Net-(Q2-C)")
+	)
+	(segment
 		(start 125 80.54)
 		(end 125 91.46)
@@
 		(layer "F.Cu")
 		(net "Net-(Q4-E)")
+	)
+	(segment
+		(start 136 98.73)
+		(end 142.19 98.73)
+		(width 0.2)
+		(layer "F.Cu")
+		(net "Net-(J_LC1-A)")
+	)
+	(segment
+		(start 142.19 98.73)
+		(end 142.46 99)
+		(width 0.2)
+		(layer "F.Cu")
+		(net "Net-(J_LC1-A)")
 	)
 	(segment
@@
 		(width 0.2)
 		(layer "F.Cu")
+		(net "Net-(U2A-+)")
+	)
+	(segment
+		(start 182 112.88)
+		(end 182 110.62)
+		(width 0.2)
+		(layer "F.Cu")
