File: Checkpoint 2/KiCAD/Diseño_v2/Diseño_v2.kicad_pcb (KiCad board)
At the start: 2 copper layers, 160 x 125 mm, 43 parts, among them J1 Conn_01x02, J2 Conn_01x02, J3 Conn_01x03, Q1 BC547, Q2 BC547, Q3 BC557, Q4 BC557, Q5 BC547, Q6 TIP32A, Q7 BC547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

Commit message: Corregí el esquemático y generé los archivos de fabricación
Parts:
- added C_COMP2: 100n, Capacitor_THT:C_Disc_D5.0mm_W2.5mm_P2.50mm, F.Cu at (170.8, 89.2)
- added R_COMP2: 100, Resistor_THT:R_Axial_DIN0207_L6.3mm_D2.5mm_P7.62mm_Horizontal, F.Cu at (175.2, 81.6)
Routing:
- net GND: track 215.6 -> 242.3 mm
- net Net-(C_COMP2-Pad1): track 0.00 -> 4.50 mm
- net /Vf: track 39.8 -> 43.5 mm

Commit message: Actualicé el PCB
Parts:
- removed C_COMP2: 100n, Capacitor_THT:C_Disc_D5.0mm_W2.5mm_P2.50mm
- removed R_COMP2: 100, Resistor_THT:R_Axial_DIN0207_L6.3mm_D2.5mm_P7.62mm_Horizontal
- C_COMP1: value 68n -> 330n
- R_COMP1: value 100 -> 22
Routing:
- net GND: track 242.3 -> 215.6 mm
- net Net-(C_COMP2-Pad1): track 4.50 -> 0.00 mm
- net /Vf: track 43.5 -> 39.8 mm
