File: Checkpoint 2/KiCAD/Diseño_v3/Diseño_v3.kicad_pcb (KiCad board)
At the start: 2 copper layers, 160 x 110 mm, 53 parts, among them J1 Conn_01x02, J2 Conn_01x02, Q1 BC547, Q2 BC547, Q3 BC557, Q4 BC557, Q5 BC547, Q6 TIP32A, Q7 BC547, Q8 BC547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

Commit message: últimos retoques al PCB
Other:
- board text added: "GND"
- board text added: "Grupo 5 - DCE - 1C2026 García Vitale Cabrera Moya"
- board text added: "Vreg"

Commit message: archivos gerber
Routing:
- net /Vref: track 156.0 -> 221.5 mm
