File: Checkpoint 3/KiCad/Diseño_v3/Diseño_v3.kicad_pcb (KiCad board)
At the start: 2 copper layers, 160 x 110 mm, 53 parts, among them J1 Conn_01x02, J2 Conn_01x02, Q1 BC547, Q2 BC547, Q3 BC557, Q4 BC557, Q5 BC547, Q6 TIP32A, Q7 BC547, Q8 BC547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

Commit message: Arreglando la placa
Parts:
- Rx1: value 10k -> 3k9
- Rx2: value 3k9 -> 10k
Changed lines of the file:
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@@
 			)
 		)
-		(property "Value" "10k"
+		(property "Value" "3k9"
 			(at 3.81 2.37 0)
 			(layer "F.Fab")
@@
 			)
 		)
-		(property "Value" "3k9"
+		(property "Value" "10k"
 			(at 3.81 2.37 90)
 			(layer "F.Fab")
