File: Checkpoint 3/KiCad/Diseño_v3/Diseño_v3.kicad_sch (KiCad schematic)
At the start: 49 parts, among them J1 Conn_01x02, J2 Conn_01x02, Q1 BC547, Q2 BC547, Q3 BC557, Q4 BC557, Q5 BC547, Q6 TIP32A, Q7 BC547, Q8 BC547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

Commit message: Arreglando la placa
Parts:
- Rx1: value 10k -> 3k9
- Rx2: value 3k9 -> 10k
