File: Checkpoint 3/KiCad/Diseño_v4/Diseño_v4.kicad_sch (KiCad schematic)
At the start: 51 parts, among them J1 Conn_01x02, J2 Conn_01x02, Q1 BC547, Q2 BC547, Q3 BC557, Q4 BC557, Q5 BC547, Q6 TIP32A, Q7 BC547, Q8 BC547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

Commit message: corrección pcb
Parts:
- removed TP_GND1, TP_GND2, TP_LC1, TP_Out_PD1, TP_Out_f1, TP_Vref1, Vreg1: (no value), Connector_PinHeader_2.54mm:PinHeader_1x01_P2.54mm_Vertical, symbol Connector:TestPoint
- added J_LC2, J_QD1: (no value), TestPoint:TestPoint_2Pads_Pitch2.54mm_Drill0.8mm, symbol Jumper:Jumper_2_Bridged
- added R_LC3: 3k9, Resistor_THT:R_Axial_DIN0207_L6.3mm_D2.5mm_P7.62mm_Horizontal, symbol Device:R
- R_LC2: renamed from R_pull_down1; value R -> 1k
- renumbered J_Vref2 to J_LC1
Connections:
- net Vf: now also J_LC2.1 (A); no longer J_LC1.2 (B)
- net at Rf1.2, U2.1: now also R_LC3.1; no longer J_LC1.1 (A), R_LC2.1
- new net: J_LC2.2 (B), R_LC2.1, R_LC3.2
- new net: J_LC1.1 (A), Q9.1 (C)
- new net: C_COMP1.2, J_LC1.2 (B), J_QD1.2 (B), Q5.2 (B)
- new net: J_QD1.1 (A), Q2.1 (C), Q4.1 (C)
Other:
- moved on the sheet: J_LC1, Q9, R_LC2
